Commit message: add lidar, change reward function

File: gym_pybullet_drones/assets/box.urdf (robot description, URDF)
Before this commit: robot test.urdf, 1 links, 0 joints
Links:
- link baseLink: mass .1 -> 1.0; geometry collision box size=0.5 0.2 0.1; visual box size=0.5 0.2 0.1

File: gym_pybullet_drones/assets/box_obstacle.urdf (robot description, URDF)
Before this commit: robot box_obstacle, 1 links, 0 joints
Links:
- removed link box
- added link baseLink, mass 0; collision box size=1 0.2 1; visual box size=1 0.2 1
